File: pcbFiles/BuckConverterRev1.sch (KiCad schematic (older format))
At the start: 7 parts, among them U7 TPS63001DRCT

Commit message: Update Footprints and Board Layers
Still need to get foorprint for x... device and the lpf may need to make them if I cannot find them @willcarroll7
Parts:
- C35, C36, C37, C38: footprint (none) -> Capacitors_SMD:C_0402
- L5: footprint (none) -> Inductors_SMD:L_0603
- R15: footprint (none) -> Resistors_SMD:R_0402
- U7: footprint SON50P300X300X100-11N -> TPS63001DRCT:SON50P300X300X100-11N
Changed lines of the file:
@@
-EESchema Schematic File Version 4
+EESchema Schematic File Version 2
 LIBS:power
+LIBS:device
+LIBS:switches
+LIBS:relays
+LIBS:motors
+LIBS:transistors
+LIBS:conn
+LIBS:linear
+LIBS:regul
 LIBS:74xx
+LIBS:cmos4000
+LIBS:adc-dac
+LIBS:memory
+LIBS:xilinx
+LIBS:microcontrollers
+LIBS:dsp
+LIBS:microchip
+LIBS:analog_switches
+LIBS:motorola
+LIBS:texas
+LIBS:intel
+LIBS:audio
+LIBS:interface
+LIBS:digital-audio
+LIBS:philips
+LIBS:display
+LIBS:cypress
+LIBS:siliconi
+LIBS:opto
+LIBS:atmel
+LIBS:contrib
+LIBS:valves
+LIBS:ADS1115IDGST
+LIBS:CYW20719B1KUMLG
+LIBS:LSM9DS1TR
+LIBS:TPS63001DRCT
+LIBS:MCP73831T-2ACI_OT
+LIBS:A-1JB
+LIBS:XC6119N16A7R-G
 LIBS:GolfGloveMainBoardV1.0.0-cache
-EELAYER 26 0
+EELAYER 25 0
 EELAYER END
 $Descr A4 11693 8268
@@
 F 0 "U7" H 5069 3852 50  0000 L BNN
 F 1 "TPS63001DRCT" H 5088 1976 50  0000 L BNN
-F 2 "SON50P300X300X100-11N" H 5250 3050 50  0001 L BNN
+F 2 "TPS63001DRCT:SON50P300X300X100-11N" H 5250 3050 50  0001 L BNN
 F 3 "VSON-10 Texas Instruments" H 5250 3050 50  0001 L BNN
 F 4 "TPS63001DRCT" H 5250 3050 50  0001 L BNN "Field4"
@@
 F 0 "L5" V 4325 3300 50  0000 C CNN
 F 1 "L" V 4450 3300 50  0000 C CNN
-F 2 "" H 4375 3300 50  0001 C CNN
+F 2 "Inductors_SMD:L_0603" H 4375 3300 50  0001 C CNN
 F 3 "" H 4375 3300 50  0001 C CNN
 	1    4375 3300
@@
 F 0 "C36" H 4250 2950 50  0000 L CNN
 F 1 "C" H 4250 2750 50  0000 L CNN
-F 2 "" H 4263 2700 50  0001 C CNN
+F 2 "Capacitors_SMD:C_0402" H 4263 2700 50  0001 C CNN
 F 3 "" H 4225 2850 50  0001 C CNN
 	1    4225 2850
@@
 F 0 "C35" H 3900 2800 50  0000 L CNN
 F 1 "C" H 3900 2600 50  0000 L CNN
-F 2 "" H 3913 2550 50  0001 C CNN
+F 2 "Capacitors_SMD:C_0402" H 3913 2550 50  0001 C CNN
 F 3 "" H 3875 2700 50  0001 C CNN
 	1    3875 2700
@@
 F 0 "C37" H 6125 2800 50  0000 L CNN
 F 1 "C" H 6125 2600 50  0000 L CNN
-F 2 "" H 6138 2550 50  0001 C CNN
+F 2 "Capacitors_SMD:C_0402" H 6138 2550 50  0001 C CNN
 F 3 "" H 6100 2700 50  0001 C CNN
 	1    6100 2700
@@
 F 0 "C38" H 6375 2800 50  0000 L CNN
 F 1 "C" H 6375 2600 50  0000 L CNN
-F 2 "" H 6388 2550 50  0001 C CNN
+F 2 "Capacitors_SMD:C_0402" H 6388 2550 50  0001 C CNN
 F 3 "" H 6350 2700 50  0001 C CNN
 	1    6350 2700
@@
 F 0 "R15" V 4530 2700 50  0000 C CNN
 F 1 "R" V 4450 2700 50  0000 C CNN
-F 2 "" V 4380 2700 50  0001 C CNN
+F 2 "Resistors_SMD:R_0402" V 4380 2700 50  0001 C CNN
 F 3 "" H 4450 2700 50  0001 C CNN
 	1    4450 2700

Commit message: Ready For Review
Parts:
- added F1: Polyfuse, Resistors_SMD:R_0603_HandSoldering, symbol Polyfuse
Connections:
- net BuckOut: now also F1.1; no longer C37.1, C38.1, U7.1 (VOUT), U7.10 (FB)
- new net: C37.1, C38.1, F1.2, U7.1 (VOUT), U7.10 (FB)
Changed lines of the file:
@@
 	4550 3450 4550 3350
 Wire Wire Line
-	5950 2550 6525 2550
+	5950 2550 6625 2550
 Connection ~ 6100 2550
 Wire Wire Line
@@
 Wire Wire Line
 	5950 2950 5950 2550
-Text HLabel 6525 2550 2    60   Input ~ 0
+Text HLabel 7075 2550 2    60   Input ~ 0
 BuckOut
 Connection ~ 6350 2550
+$Comp
+L Polyfuse F1
+U 1 1 5CAEC441
+P 6775 2550
+F 0 "F1" V 6675 2550 50  0000 C CNN
+F 1 "Polyfuse" V 6875 2550 50  0000 C CNN
+F 2 "Resistors_SMD:R_0603_HandSoldering" H 6825 2350 50  0001 L CNN
+F 3 "" H 6775 2550 50  0001 C CNN
+	1    6775 2550
+	0    1    1    0
+$EndComp
+Wire Wire Line
+	7075 2550 6925 2550
 $EndSCHEMATC
