File: pcbFiles/GolfGloveMainBoardV1.0.0.sch (KiCad schematic (older format))
At the start: 35 parts, among them J1 USB_C_Receptacle, J11 Conn_01x16_Male, J12 HOST_WAKE, J13 TP4, J17 Conn_01x02, J2 Conn_01x06, J3 USB_C_Receptacle, J4 Conn_01x01, J5 Conn_01x01, SW1 SW_SPDT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

Commit message: Update Board Files
Updated schematic files, completed REV1.0 of the board design, waiting for review by @willcarroll7
Parts:
- removed J4, J5: Conn_01x01, Wire_Pads:SolderWirePad_single_2mmDrill, symbol Conn_01x01
Connections:
- wire segments 201 -> 233
Other:
- moved on the sheet: J11, SW1

Commit message: Updates
Parts:
- removed L1, L6: L, Inductors_SMD:L_0402, symbol L
- removed Y2: Crystal_GND23, Crystals:Crystal_SMD_0603-4pin_6.0x3.5mm_HandSoldering, symbol Crystal_GND23
- added C19, C20: C, Capacitors_SMD:C_0402, symbol C
- added Y3: Crystal_GND24, Crystals:Crystal_SMD_0603-4pin_6.0x3.5mm_HandSoldering, symbol Crystal_GND24
Connections:
- net labels removed: VBAT
- wire segments 233 -> 241
Changed lines of the file:
@@
 Text Notes 7525 4400 0    60   ~ 0
 8.2pf
-$Comp
-L Crystal_GND23 Y2
-U 1 1 5C45C3BB
-P 7650 4975
-F 0 "Y2" H 7775 5175 50  0000 L CNN
-F 1 "Crystal_GND23" H 6675 4975 50  0000 L CNN
-F 2 "Crystals:Crystal_SMD_0603-4pin_6.0x3.5mm_HandSoldering" H 7650 4975 50  0001 C CNN
-F 3 "" H 7650 4975 50  0001 C CNN
-	1    7650 4975
-	-1   0    0    1
-$EndComp
 Text GLabel 7550 4775 0    60   Input ~ 0
 GND
@@
 GND
 Text GLabel 7150 3225 0    60   Input ~ 0
-VBAT
+3.3v
 $Comp
 L C C22
@@
 	-1   0    0    1
 $EndComp
-$Comp
-L L L1
-U 1 1 5C59D98B
-P 6625 4525
-F 0 "L1" V 6575 4525 50  0000 C CNN
-F 1 "L" V 6700 4525 50  0000 C CNN
-F 2 "Inductors_SMD:L_0402" H 6625 4525 50  0001 C CNN
-F 3 "" H 6625 4525 50  0001 C CNN
-	1    6625 4525
-	0    1    1    0
-$EndComp
-$Comp
-L L L6
-U 1 1 5C59DAC4
-P 6850 4325
-F 0 "L6" V 6800 4325 50  0000 C CNN
-F 1 "L" V 6925 4325 50  0000 C CNN
-F 2 "Inductors_SMD:L_0402" H 6850 4325 50  0001 C CNN
-F 3 "" H 6850 4325 50  0001 C CNN
-	1    6850 4325
-	1    0    0    -1
-$EndComp
 Text GLabel 6775 4100 0    60   Input ~ 0
 GND
@@
 	8900 4025 9025 4025
 Connection ~ 9850 4925
+$Comp
+L Crystal_GND24 Y3
+U 1 1 5C99C2D0
+P 7650 4975
+F 0 "Y3" H 7775 5175 50  0000 L CNN
+F 1 "Crystal_GND24" H 7775 5100 50  0000 L CNN
+F 2 "Crystals:Crystal_SMD_0603-4pin_6.0x3.5mm_HandSoldering" H 7650 4975 50  0001 C CNN
+F 3 "" H 7650 4975 50  0001 C CNN
+	1    7650 4975
+	1    0    0    -1
+$EndComp
+$Comp
+L C C19
+U 1 1 5C9FB833
+P 6625 4525
+F 0 "C19" H 6650 4625 50  0000 L CNN
+F 1 "C" H 6650 4425 50  0000 L CNN
+F 2 "Capacitors_SMD:C_0402" H 6663 4375 50  0001 C CNN
+F 3 "" H 6625 4525 50  0001 C CNN
+	1    6625 4525
+	0    1    1    0
+$EndComp
+$Comp
+L C C20
+U 1 1 5C9FB984
+P 6850 4325
+F 0 "C20" H 6875 4425 50  0000 L CNN
+F 1 "C" H 6875 4225 50  0000 L CNN
+F 2 "Capacitors_SMD:C_0402" H 6888 4175 50  0001 C CNN
+F 3 "" H 6850 4325 50  0001 C CNN
+	1    6850 4325
+	1    0    0    -1
+$EndComp
+Wire Wire Line
+	9850 4725 9850 4650
+Wire Wire Line
+	9850 4650 9375 4650
+Wire Wire Line
+	9375 4650 9375 4575
+Wire Wire Line
+	9375 4575 9325 4575
+Wire Wire Line
+	9325 4725 9550 4725
+Wire Wire Line
+	9550 4725 9550 4800
+Wire Wire Line
+	9550 4800 9850 4800
+Wire Wire Line
+	9850 4800 9850 4825
 $EndSCHEMATC

Commit message: Remove Headers
Parts:
- removed J12: HOST_WAKE, Pin_Headers:Pin_Header_Straight_1x01_Pitch2.54mm, symbol Conn_01x01
- removed J13: TP4, Pin_Headers:Pin_Header_Straight_1x01_Pitch2.54mm, symbol Conn_01x01
Changed lines of the file:
@@
 Text GLabel 7850 2925 2    60   Input ~ 0
 CBUCK_OUT
-$Comp
-L Conn_01x01 J13
-U 1 1 5C47519F
-P 10775 1975
-F 0 "J13" H 10775 2075 50  0000 C CNN
-F 1 "TP4" H 10775 1875 50  0000 C CNN
-F 2 "Pin_Headers:Pin_Header_Straight_1x01_Pitch2.54mm" H 10775 1975 50  0001 C CNN
-F 3 "" H 10775 1975 50  0001 C CNN
-	1    10775 1975
-	1    0    0    -1
-$EndComp
-$Comp
-L Conn_01x01 J12
-U 1 1 5C475EAA
-P 10075 2650
-F 0 "J12" H 10075 2750 50  0000 C CNN
-F 1 "HOST_WAKE" H 10075 2550 50  0000 C CNN
-F 2 "Pin_Headers:Pin_Header_Straight_1x01_Pitch2.54mm" H 10075 2650 50  0001 C CNN
-F 3 "" H 10075 2650 50  0001 C CNN
-	1    10075 2650
-	1    0    0    -1
-$EndComp
 Text Notes 10025 2000 0    60   ~ 0
 .1uf
@@
 	7850 2925 7850 3025
 Wire Wire Line
-	9850 1925 10100 1925
-Wire Wire Line
-	10100 1925 10100 1975
-Wire Wire Line
-	10100 1975 10575 1975
-Wire Wire Line
-	9850 2725 9850 2650
-Wire Wire Line
-	9850 2650 9875 2650
-Wire Wire Line
 	9325 3425 10125 3425

Commit message: Updates
Parts:
- removed J11: Conn_01x16_Male, Pin_Headers:Pin_Header_Straight_2x08_Pitch2.54mm, symbol Conn_01x16_Male
- added J4, J5, J6: Conn_01x02_Male, Pin_Headers:Pin_Header_Straight_1x02_Pitch2.54mm, symbol Conn_01x02_Male
- added SW3: SW_Push_Dual, Buttons_Switches_THT:SW_PUSH_6mm, symbol SW_Push_Dual
- Y1: footprint Crystals:Crystal_SMD_0603-2pin_6.0x3.5mm_HandSoldering -> Crystals:Crystal_SMD_3215-2pin_3.2x1.5mm
- Y3: footprint Crystals:Crystal_SMD_0603-4pin_6.0x3.5mm_HandSoldering -> Crystals:Crystal_SMD_2016-4pin_2.0x1.6mm
Connections:
- net BT_UART_CTS: now also SW3.2, SW3.4
- net GND: now also J4.2 (Pin_2), SW3.1, SW3.3
- net SCLK: now also J6.2 (Pin_2)
- net SDA: now also J6.1 (Pin_1)
- net at U4.5 (P34): now also J5.1 (Pin_1)
- net at U4.9 (P33): now also J5.2 (Pin_2)
- net at SW1.2 (B): now also J4.1 (Pin_1)
Changed lines of the file:
@@
 F 0 "Y1" H 7575 2725 50  0000 C CNN
 F 1 "Crystal" H 7575 2425 50  0000 C CNN
-F 2 "Crystals:Crystal_SMD_0603-2pin_6.0x3.5mm_HandSoldering" H 7575 2575 50  0001 C CNN
+F 2 "Crystals:Crystal_SMD_3215-2pin_3.2x1.5mm" H 7575 2575 50  0001 C CNN
 F 3 "" H 7575 2575 50  0001 C CNN
 	1    7575 2575
@@
 Text Notes 7825 4900 0    60   ~ 0
 24.000Mhz
-$Comp
-L Conn_01x16_Male J11
-U 1 1 5C4824CB
-P 9125 4125
-F 0 "J11" H 9125 4925 50  0000 C CNN
-F 1 "Conn_01x16_Male" H 9125 3225 50  0000 C CNN
-F 2 "Pin_Headers:Pin_Header_Straight_2x08_Pitch2.54mm" H 9125 4125 50  0001 C CNN
-F 3 "" H 9125 4125 50  0001 C CNN
-	1    9125 4125
-	1    0    0    -1
-$EndComp
 Text GLabel 7775 2825 0    60   Input ~ 0
 RST_N
@@
 Connection ~ 1125 3850
 Wire Wire Line
-	9425 5600 9650 5600
+	8950 5600 9650 5600
 Wire Wire Line
 	10050 5700 10125 5700
@@
 	9850 5125 9925 5125
 Wire Wire Line
-	9400 4325 9925 4325
-Wire Wire Line
-	9450 4625 9925 4625
-Wire Wire Line
 	6775 4525 7850 4525
 Wire Wire Line
@@
 	7850 2925 7850 3025
 Wire Wire Line
-	9325 3425 10125 3425
-Wire Wire Line
 	10125 3425 10125 3775
 Wire Wire Line
@@
 Wire Wire Line
 	10100 3800 10100 3525
-Wire Wire Line
-	10100 3525 9325 3525
-Wire Wire Line
-	9425 4525 10400 4525
 Wire Wire Line
 	10400 4525 10400 3750
@@
 Connection ~ 9850 3425
 Connection ~ 9850 3525
-Wire Wire Line
-	9375 4125 9925 4125
 Connection ~ 9850 4325
-Wire Wire Line
-	9850 4425 9475 4425
 Connection ~ 9850 4525
 Connection ~ 9850 4625
@@
 	6375 4525 6475 4525
 Wire Wire Line
-	9375 4225 9950 4225
-Wire Wire Line
 	3825 2250 3900 2250
 Wire Wire Line
@@
 Wire Wire Line
 	3900 2950 3825 2950
-Wire Wire Line
-	9325 3625 9425 3625
-Wire Wire Line
-	9425 3625 9425 4525
-Wire Wire Line
-	9375 4125 9375 3725
-Wire Wire Line
-	9375 3725 9325 3725
-Wire Wire Line
-	9400 4325 9400 3825
-Wire Wire Line
-	9400 3825 9325 3825
-Wire Wire Line
-	9450 4625 9450 3925
-Wire Wire Line
-	9450 3925 9325 3925
-Wire Wire Line
-	9450 3625 9450 3575
-Wire Wire Line
-	9450 3575 9325 3575
-Wire Wire Line
-	9325 3575 9325 4025
-Wire Wire Line
-	9475 3725 9475 3675
-Wire Wire Line
-	9475 3675 9050 3675
-Wire Wire Line
-	9050 3675 9050 4125
-Wire Wire Line
-	9050 4125 9325 4125
-Wire Wire Line
-	9450 3825 9450 3775
-Wire Wire Line
-	9450 3775 9075 3775
-Wire Wire Line
-	9075 3775 9075 4225
-Wire Wire Line
-	9075 4225 9325 4225
-Wire Wire Line
-	9475 3925 9475 3900
-Wire Wire Line
-	9475 3900 9100 3900
-Wire Wire Line
-	9100 3900 9100 4325
-Wire Wire Line
-	9100 4325 9325 4325
-Wire Wire Line
-	9025 4025 9025 4425
-Wire Wire Line
-	9025 4425 9325 4425
-Wire Wire Line
-	9375 4225 9375 4525
-Wire Wire Line
-	9375 4525 9325 4525
-Wire Wire Line
-	9475 4425 9475 4575
-Wire Wire Line
-	9325 4575 9325 4625
-Text GLabel 8975 4825 0    60   Input ~ 0
-GND
-Wire Wire Line
-	9325 4825 8975 4825
-Wire Wire Line
-	9325 4925 9425 4925
-Wire Wire Line
-	9425 4925 9425 5600
+Text GLabel 8850 5425 0    60   Input ~ 0
+GND
 Text GLabel 1975 2925 2    60   Input ~ 0
 PSensor2
@@
 PSensor1
 Wire Wire Line
-	9475 4925 10225 4925
-Wire Wire Line
 	10225 4925 10225 4950
 Wire Wire Line
@@
 	9950 4150 9950 4225
 Connection ~ 9850 4225
+Connection ~ 9850 4925
+$Comp
+L Crystal_GND24 Y3
+U 1 1 5C99C2D0
+P 7650 4975
+F 0 "Y3" H 7775 5175 50  0000 L CNN
+F 1 "Crystal_GND24" H 7775 5100 50  0000 L CNN
+F 2 "Crystals:Crystal_SMD_2016-4pin_2.0x1.6mm" H 7650 4975 50  0001 C CNN
+F 3 "" H 7650 4975 50  0001 C CNN
+	1    7650 4975
+	1    0    0    -1
+$EndComp
+$Comp
+L C C19
+U 1 1 5C9FB833
+P 6625 4525
+F 0 "C19" H 6650 4625 50  0000 L CNN
+F 1 "C" H 6650 4425 50  0000 L CNN
+F 2 "Capacitors_SMD:C_0402" H 6663 4375 50  0001 C CNN
+F 3 "" H 6625 4525 50  0001 C CNN
+	1    6625 4525
+	0    1    1    0
+$EndComp
+$Comp
+L C C20
+U 1 1 5C9FB984
+P 6850 4325
+F 0 "C20" H 6875 4425 50  0000 L CNN
+F 1 "C" H 6875 4225 50  0000 L CNN
+F 2 "Capacitors_SMD:C_0402" H 6888 4175 50  0001 C CNN
+F 3 "" H 6850 4325 50  0001 C CNN
+	1    6850 4325
+	1    0    0    -1
+$EndComp
+$Comp
+L SW_Push_Dual SW3
+U 1 1 5CAD92C9
+P 4975 3100
+F 0 "SW3" H 5025 3200 50  0000 L CNN
+F 1 "SW_Push_Dual" H 4975 2830 50  0000 C CNN
+F 2 "Buttons_Switches_THT:SW_PUSH_6mm" H 4975 3300 50  0001 C CNN
+F 3 "" H 4975 3300 50  0001 C CNN
+	1    4975 3100
+	0    -1   -1   0
+$EndComp
+Wire Wire Line
+	5775 2850 5775 2650
+Wire Wire Line
+	5775 2650 5175 2650
+Wire Wire Line
+	5175 2650 5175 2900
+Connection ~ 5775 2850
+Wire Wire Line
+	5175 3300 5175 3675
+Wire Wire Line
+	5175 3675 5675 3675
+Wire Wire Line
+	5675 3675 5675 3375
+Wire Wire Line
+	5675 3375 5775 3375
+Wire Wire Line
+	5775 3375 5775 3350
+Connection ~ 5775 3350
+Wire Wire Line
+	5175 2900 4975 2900
+Wire Wire Line
+	4975 3300 5175 3300
 $Comp
 L CYW20719B1KUMLG U4
@@
 	1    0    0    -1
 $EndComp
-Wire Wire Line
-	9475 4925 9475 4775
-Wire Wire Line
-	9475 4775 9025 4775
-Wire Wire Line
-	9025 4775 9025 4500
-Wire Wire Line
-	9025 4500 8900 4500
-Wire Wire Line
-	8900 4500 8900 4025
-Wire Wire Line
-	8900 4025 9025 4025
-Connection ~ 9850 4925
-$Comp
-L Crystal_GND24 Y3
-U 1 1 5C99C2D0
-P 7650 4975
-F 0 "Y3" H 7775 5175 50  0000 L CNN
-F 1 "Crystal_GND24" H 7775 5100 50  0000 L CNN
-F 2 "Crystals:Crystal_SMD_0603-4pin_6.0x3.5mm_HandSoldering" H 7650 4975 50  0001 C CNN
-F 3 "" H 7650 4975 50  0001 C CNN
-	1    7650 4975
-	1    0    0    -1
-$EndComp
-$Comp
-L C C19
-U 1 1 5C9FB833
-P 6625 4525
-F 0 "C19" H 6650 4625 50  0000 L CNN
-F 1 "C" H 6650 4425 50  0000 L CNN
-F 2 "Capacitors_SMD:C_0402" H 6663 4375 50  0001 C CNN
-F 3 "" H 6625 4525 50  0001 C CNN
-	1    6625 4525
-	0    1    1    0
-$EndComp
-$Comp
-L C C20
-U 1 1 5C9FB984
-P 6850 4325
-F 0 "C20" H 6875 4425 50  0000 L CNN
-F 1 "C" H 6875 4225 50  0000 L CNN
-F 2 "Capacitors_SMD:C_0402" H 6888 4175 50  0001 C CNN
-F 3 "" H 6850 4325 50  0001 C CNN
-	1    6850 4325
-	1    0    0    -1
-$EndComp
-Wire Wire Line
-	9850 4725 9850 4650
-Wire Wire Line
-	9850 4650 9375 4650
-Wire Wire Line
-	9375 4650 9375 4575
-Wire Wire Line
-	9375 4575 9325 4575
-Wire Wire Line
-	9325 4725 9550 4725
-Wire Wire Line
-	9550 4725 9550 4800
-Wire Wire Line
-	9550 4800 9850 4800
-Wire Wire Line
-	9850 4800 9850 4825
+$Comp
+L Conn_01x02_Male J6
+U 1 1 5CAE13FE
+P 10850 4575
+F 0 "J6" H 10850 4675 50  0000 C CNN
+F 1 "Conn_01x02_Male" H 10850 4375 50  0000 C CNN
+F 2 "Pin_Headers:Pin_Header_Straight_1x02_Pitch2.54mm" H 10850 4575 50  0001 C CNN
+F 3 "" H 10850 4575 50  0001 C CNN
+	1    10850 4575
+	-1   0    0    1
+$EndComp
+Wire Wire Line
+	9850 4325 10650 4325
+Wire Wire Line
+	10650 4325 10650 4475
+Wire Wire Line
+	9850 4625 10650 4625
+Wire Wire Line
+	10650 4625 10650 4575
+$Comp
+L Conn_01x02_Male J5
+U 1 1 5CAE37EF
+P 10175 4825
+F 0 "J5" H 10175 4925 50  0000 C CNN
+F 1 "Conn_01x02_Male" H 10175 4625 50  0000 C CNN
+F 2 "Pin_Headers:Pin_Header_Straight_1x02_Pitch2.54mm" H 10175 4825 50  0001 C CNN
+F 3 "" H 10175 4825 50  0001 C CNN
+	1    10175 4825
+	-1   0    0    1
+$EndComp
+Wire Wire Line
+	9975 4725 9850 4725
+Wire Wire Line
+	9850 4825 9975 4825
+Wire Wire Line
+	9850 4925 10225 4925
+Wire Wire Line
+	9925 4125 9850 4125
+Wire Wire Line
+	9950 4225 9850 4225
+Wire Wire Line
+	10400 4525 9850 4525
+Wire Wire Line
+	10100 3525 9850 3525
+Wire Wire Line
+	9850 3425 10125 3425
+$Comp
+L Conn_01x02_Male J4
+U 1 1 5CAE6E60
+P 9150 5525
+F 0 "J4" H 9150 5625 50  0000 C CNN
+F 1 "Conn_01x02_Male" H 9150 5325 50  0000 C CNN
+F 2 "Pin_Headers:Pin_Header_Straight_1x02_Pitch2.54mm" H 9150 5525 50  0001 C CNN
+F 3 "" H 9150 5525 50  0001 C CNN
+	1    9150 5525
+	-1   0    0    1
+$EndComp
+Wire Wire Line
+	8950 5600 8950 5525
+Wire Wire Line
+	8850 5425 8950 5425
 $EndSCHEMATC

Commit message: Ready For Review
Parts:
- added R14, R16: R, Resistors_SMD:R_0402, symbol R
Connections:
- net 3.3v: now also J1.A8 (SBU1), J1.B8 (SBU2); no longer J1.A2 (TX1+), J1.A3 (TX1-), J1.B2 (TX2+), J1.B3 (TX2-)
- net GND: now also R14.1, R16.1
- net PSensor1: now also J1.A11 (RX2+), J1.B11 (RX1+), J3.A11 (RX2+), J3.B11 (RX1+); no longer J1.A10 (RX2-), J3.A10 (RX2-), J3.B10 (RX1-)
- net PSensor2: now also J1.A2 (TX1+), J1.B2 (TX2+), J3.A2 (TX1+), J3.B2 (TX2+); no longer J1.A11 (RX2+), J3.A11 (RX2+), J3.B11 (RX1+)
- net SCLK: now also J1.A3 (TX1-), J1.B3 (TX2-); no longer J1.A6 (D+), J1.B6 (D+)
- net SCLK-USB: now also J3.A3 (TX1-), J3.B3 (TX2-); no longer J3.A6 (D+), J3.B6 (D+)
- net SDA: now also J1.A10 (RX2-), J1.B10 (RX1-); no longer J1.A7 (D-), J1.B7 (D-)
- net SDA-USB: now also J3.A10 (RX2-), J3.B10 (RX1-); no longer J3.A7 (D-), J3.B7 (D-)
- net USBVCC: now also J3.A8 (SBU1), J3.B8 (SBU2); no longer J3.A2 (TX1+), J3.A3 (TX1-), J3.B2 (TX2+), J3.B3 (TX2-)
- net at J1.A5 (CC1): now also R14.2
- net at J1.B5 (CC2): now also R16.2
Other:
- note added: "56k"
Changed lines of the file:
@@
 	1    0    0    -1
 $EndComp
-Text GLabel 3875 3150 2    60   Input ~ 0
-USBVCC
-Text GLabel 3900 1950 2    60   Input ~ 0
-SCLK-USB
-Text GLabel 3900 1850 2    60   Input ~ 0
-SDA-USB
 Text GLabel 3400 3875 2    60   Input ~ 0
 USBGND
-Text GLabel 2000 1925 2    60   Input ~ 0
+Text GLabel 2000 2525 2    60   Input ~ 0
 SCLK
-Text GLabel 2000 1825 2    60   Input ~ 0
+Text GLabel 1975 2225 2    60   Input ~ 0
 SDA
 Text GLabel 1950 825  2    60   Input ~ 0
@@
 Text GLabel 10125 5500 2    60   Input ~ 0
 BatteryOutChg
-Text GLabel 1975 3125 2    60   Input ~ 0
+Text GLabel 2000 3425 2    60   Input ~ 0
 3.3v
-Text GLabel 1975 3225 2    60   Input ~ 0
-3.3v
-Text GLabel 3875 3250 2    60   Input ~ 0
-USBVCC
 $Comp
 L Crystal Y1
@@
 PSensor2
 Text GLabel 5900 6900 2    60   Input ~ 0
-PSensor1
-Text GLabel 3900 2350 2    60   Input ~ 0
-PSensor2
-Text GLabel 3900 2250 2    60   Input ~ 0
 PSensor1
 Text GLabel 9925 4325 2    60   Input ~ 0
@@
 Text GLabel 7775 2825 0    60   Input ~ 0
 RST_N
-Text GLabel 1975 2525 2    60   Input ~ 0
-3.3v
-Text GLabel 1975 2625 2    60   Input ~ 0
-3.3v
-Text GLabel 3875 2550 2    60   Input ~ 0
-USBVCC
-Text GLabel 3875 2650 2    60   Input ~ 0
-USBVCC
 $Sheet
 S 1475 7300 775  350
@@
 Text GLabel 6775 4100 0    60   Input ~ 0
 GND
-Text GLabel 3900 2950 2    60   Input ~ 0
-PSensor2
-Text GLabel 3900 2850 2    60   Input ~ 0
-PSensor1
-Wire Wire Line
-	3900 1850 3825 1850
-Wire Wire Line
-	3900 1850 3900 1750
-Wire Wire Line
-	3900 1750 3825 1750
-Wire Wire Line
-	3900 1950 3825 1950
-Wire Wire Line
-	3900 1950 3900 2050
-Wire Wire Line
-	3900 2050 3825 2050
 Wire Wire Line
 	2925 3875 3400 3875
@@
 Connection ~ 3025 3875
 Wire Wire Line
-	1925 1825 2000 1825
-Wire Wire Line
-	1925 1925 2000 1925
-Wire Wire Line
-	1950 1925 1950 2025
-Wire Wire Line
-	1950 2025 1925 2025
-Connection ~ 1950 1925
-Wire Wire Line
-	1950 1825 1950 1725
-Wire Wire Line
-	1950 1725 1925 1725
-Connection ~ 1950 1825
-Wire Wire Line
 	1950 825  1950 1225
 Wire Wire Line
@@
 	10050 5500 10125 5500
 Wire Wire Line
-	1975 3125 1925 3125
-Wire Wire Line
-	1925 3225 1975 3225
-Wire Wire Line
-	3825 3150 3875 3150
-Wire Wire Line
-	3875 3250 3825 3250
+	1925 3125 2000 3125
+Wire Wire Line
+	1925 3225 2000 3225
 Wire Wire Line
 	7450 2075 7375 2075
@@
 Connection ~ 9850 4125
 Wire Wire Line
-	1975 2525 1925 2525
-Wire Wire Line
-	1925 2625 1975 2625
-Wire Wire Line
-	3825 2550 3875 2550
-Wire Wire Line
-	3875 2650 3825 2650
+	1925 2525 2000 2525
+Wire Wire Line
+	1925 2625 2000 2625
 Wire Wire Line
 	1350 7375 1475 7375
@@
 Wire Wire Line
 	6375 4525 6475 4525
-Wire Wire Line
-	3825 2250 3900 2250
-Wire Wire Line
-	3825 2350 3900 2350
-Wire Wire Line
-	3825 2850 3900 2850
-Wire Wire Line
-	3900 2950 3825 2950
 Text GLabel 8850 5425 0    60   Input ~ 0
 GND
-Text GLabel 1975 2925 2    60   Input ~ 0
-PSensor2
-Text GLabel 1975 2825 2    60   Input ~ 0
-PSensor1
-Wire Wire Line
-	1925 2825 1975 2825
-Wire Wire Line
-	1975 2925 1925 2925
+Wire Wire Line
+	1925 2825 2000 2825
+Wire Wire Line
+	1925 2925 2000 2925
 Text GLabel 10225 4950 2    60   Input ~ 0
 PSensor2
@@
 Wire Wire Line
 	8850 5425 8950 5425
+Text GLabel 2000 2625 2    60   Input ~ 0
+PSensor2
+Text GLabel 2000 2925 2    60   Input ~ 0
+PSensor1
+Text GLabel 2000 3525 2    60   Input ~ 0
+3.3v
+Text GLabel 2000 2825 2    60   Input ~ 0
+SDA
+Wire Wire Line
+	1975 2225 1925 2225
+Text GLabel 2000 3125 2    60   Input ~ 0
+SCLK
+Text GLabel 1975 2325 2    60   Input ~ 0
+PSensor1
+Text GLabel 2000 3225 2    60   Input ~ 0
+PSensor2
+Wire Wire Line
+	1975 2325 1925 2325
+Wire Wire Line
+	1925 1525 2075 1525
+Wire Wire Line
+	1925 1425 2075 1425
+Wire Wire Line
+	3900 2950 3825 2950
+Wire Wire Line
+	3825 2850 3900 2850
+Wire Wire Line
+	3825 2350 3900 2350
+Wire Wire Line
+	3825 2250 3900 2250
+Wire Wire Line
+	3875 2650 3825 2650
+Wire Wire Line
+	3825 2550 3875 2550
+Wire Wire Line
+	3875 3250 3825 3250
+Wire Wire Line
+	3825 3150 3875 3150
+Text GLabel 3900 2350 2    60   Input ~ 0
+PSensor1
+Text GLabel 3875 3250 2    60   Input ~ 0
+PSensor2
+Text GLabel 3900 2950 2    60   Input ~ 0
+PSensor1
+Text GLabel 3875 2650 2    60   Input ~ 0
+PSensor2
+Text GLabel 3900 3550 2    60   Input ~ 0
+USBVCC
+Text GLabel 3900 2850 2    60   Input ~ 0
+SDA-USB
+Text GLabel 3875 2550 2    60   Input ~ 0
+SCLK-USB
+Text GLabel 3900 3450 2    60   Input ~ 0
+USBVCC
+Text GLabel 3900 2250 2    60   Input ~ 0
+SDA-USB
+Text GLabel 3875 3150 2    60   Input ~ 0
+SCLK-USB
+Wire Wire Line
+	3825 3450 3900 3450
+Wire Wire Line
+	3900 3550 3825 3550
+Wire Wire Line
+	2000 3525 1925 3525
+Wire Wire Line
+	1925 3425 2000 3425
+$Comp
+L R R14
+U 1 1 5CB0636C
+P 2225 1425
+F 0 "R14" V 2305 1425 50  0000 C CNN
+F 1 "R" V 2225 1425 50  0000 C CNN
+F 2 "Resistors_SMD:R_0402" V 2155 1425 50  0001 C CNN
+F 3 "" H 2225 1425 50  0001 C CNN
+	1    2225 1425
+	0    1    1    0
+$EndComp
+$Comp
+L R R16
+U 1 1 5CB06CF2
+P 2225 1525
+F 0 "R16" V 2305 1525 50  0000 C CNN
+F 1 "R" V 2225 1525 50  0000 C CNN
+F 2 "Resistors_SMD:R_0402" V 2155 1525 50  0001 C CNN
+F 3 "" H 2225 1525 50  0001 C CNN
+	1    2225 1525
+	0    1    1    0
+$EndComp
+Text GLabel 2475 1475 2    60   Input ~ 0
+GND
+Wire Wire Line
+	2375 1425 2475 1425
+Wire Wire Line
+	2475 1425 2475 1525
+Wire Wire Line
+	2475 1525 2375 1525
+Text Notes 2150 1350 0    60   ~ 0
+56k
+Text Notes 2150 1725 0    60   ~ 0
+56k
 $EndSCHEMATC

Commit message: Add LED for Power Indication
Parts:
- added D2: LED, Capacitors_SMD:C_0603, symbol LED
- added R17: R, Resistors_SMD:R_0402, symbol R
Connections:
- net 3.3v: now also R17.2
- net GND: now also D2.1 (K)
- new net: D2.2 (A), R17.1
- no-connect marks 0 -> 1
Other:
- note added: "POOP DICK BALLS\n"
Changed lines of the file:
@@
 Text Notes 2150 1725 0    60   ~ 0
 56k
+NoConn ~ 9850 1925
+Text GLabel 1975 4400 0    60   Input ~ 0
+3.3v
+Text GLabel 2825 4400 2    60   Input ~ 0
+GND
+Text Notes 3100 4900 0    60   ~ 0
+POOP DICK BALLS\n
+$Comp
+L LED D2
+U 1 1 5CB3D009
+P 2575 4400
+F 0 "D2" H 2575 4500 50  0000 C CNN
+F 1 "LED" H 2575 4300 50  0000 C CNN
+F 2 "Capacitors_SMD:C_0603" H 2575 4400 50  0001 C CNN
+F 3 "" H 2575 4400 50  0001 C CNN
+	1    2575 4400
+	-1   0    0    1
+$EndComp
+$Comp
+L R R17
+U 1 1 5CB3D164
+P 2200 4400
+F 0 "R17" V 2280 4400 50  0000 C CNN
+F 1 "R" V 2200 4400 50  0000 C CNN
+F 2 "Resistors_SMD:R_0402" V 2130 4400 50  0001 C CNN
+F 3 "" H 2200 4400 50  0001 C CNN
+	1    2200 4400
+	0    1    1    0
+$EndComp
+Wire Wire Line
+	2825 4400 2725 4400
+Wire Wire Line
+	2425 4400 2350 4400
+Wire Wire Line
+	2050 4400 1975 4400
 $EndSCHEMATC

Commit message: Removed Humorous Text
Other:
- note removed: "POOP DICK BALLS\n"
Changed lines of the file:
@@
 Text GLabel 2825 4400 2    60   Input ~ 0
 GND
-Text Notes 3100 4900 0    60   ~ 0
-POOP DICK BALLS\n
 $Comp
 L LED D2
